File: pcb/sensors.kicad_sch (KiCad schematic)
At the start: 26 parts, among them J12 Conn_01x03, J13 Conn_01x03, J14 Conn_01x03, J15 Conn_01x03, J6 Conn_01x03, U5 AH1815-W-7, U6 AH1815-W-7, U7 AH1815-W-7, U8 AH1815-W-7, U9 AH1815-W-7

Commit message: Rework 6
Added power flags to external power inputs. Fixed Motor connector pins from Unspecified to Passive, per KiCad fashion. Made the ERC pass without exclusions.

Added power decoupling to Hall sensor connectors and to the Neopixels.

Moved the IN test point for better probing accessibility. Test points use teardrop connections for integrity in face of probing.

Added a ground clip area for scope probes etc.

Added a 3D model of the pushbuttons.
Rework 6

Change revision to 1.2.
Other:
- moved on the sheet: J13, J14
